File: pcb_files/Pacifista_ESP/Pacifistabot-ESP-01s.sch (KiCad schematic (older format))
At the start: 25 parts, among them J1 Conn_01x01, J10 Conn_01x03, J11 Conn_01x03, J2 Conn_01x01, J3 Conn_01x09, J4 Conn_01x06, J5 Conn_01x06, J6 Conn_01x06, J7 Conn_01x06, J8 Conn_01x06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

Commit message: Corrección de los pines de la PCB y el logo de DB
Parts:
- C3: symbol pspice:CAP -> Pacifistabot-ESP-01s-rescue:CAP-pspice
- J3: symbol Connector_Generic:Conn_01x09 -> Pacifistabot-ESP-01s-rescue:Conn_01x09-Connector_Generic
- J9: symbol Connector_Generic:Conn_01x06 -> Pacifistabot-ESP-01s-rescue:Conn_01x06-Connector_Generic
- R1, R2, R3, R6, R7: symbol Device:R -> Pacifistabot-ESP-01s-rescue:R-Device
- U2: symbol Regulator_Linear:AMS1117 -> Pacifistabot-ESP-01s-rescue:AMS1117-Regulator_Linear
Changed lines of the file:
@@
 EESchema Schematic File Version 4
 LIBS:Pacifistabot-ESP-01s-cache
-EELAYER 26 0
+EELAYER 30 0
 EELAYER END
 $Descr A4 11693 8268
@@
 	6250 2450 6400 2450
 $Comp
-L Device:R R2
+L Pacifistabot-ESP-01s-rescue:R-Device R2
 U 1 1 5DC3A91A
 P 6700 2350
@@
 $EndComp
 $Comp
-L Device:R R3
+L Pacifistabot-ESP-01s-rescue:R-Device R3
 U 1 1 5DC40FD8
 P 6900 2550
@@
 	2350 4650 2700 4650
 $Comp
-L Connector_Generic:Conn_01x09 J3
+L Pacifistabot-ESP-01s-rescue:Conn_01x09-Connector_Generic J3
 U 1 1 5DE0D3A4
 P 6550 3150
@@
 $EndComp
 $Comp
-L power:+3.3V #PWR0109
+L Pacifistabot-ESP-01s-rescue:+3.3V-power #PWR0109
 U 1 1 5DAF2344
 P 2750 1300
@@
 $EndComp
 $Comp
-L Device:R R1
+L Pacifistabot-ESP-01s-rescue:R-Device R1
 U 1 1 5DB02EEC
 P 3100 1400
@@
 	5300 1600 5450 1600
 $Comp
-L Regulator_Linear:AMS1117 U2
+L Pacifistabot-ESP-01s-rescue:AMS1117-Regulator_Linear U2
 U 1 1 5DB788B1
 P 2150 1400
@@
 Alimentación
 $Comp
-L Device:R R7
+L Pacifistabot-ESP-01s-rescue:R-Device R7
 U 1 1 5DEBB805
 P 7050 1500
@@
 $EndComp
 $Comp
-L Device:R R6
+L Pacifistabot-ESP-01s-rescue:R-Device R6
 U 1 1 5DEBB80B
 P 6700 1500
@@
 	7050 1250 7450 1250
 $Comp
-L pspice:CAP C3
+L Pacifistabot-ESP-01s-rescue:CAP-pspice C3
 U 1 1 5DEBB814
 P 7700 1250
@@
 5V
 $Comp
-L power:GND #PWR0112
+L Pacifistabot-ESP-01s-rescue:GND-power #PWR0112
 U 1 1 5DEBB81E
 P 6700 1800
@@
 NoConn ~ 8350 750
 $Comp
-L Connector_Generic:Conn_01x06 J9
+L Pacifistabot-ESP-01s-rescue:Conn_01x06-Connector_Generic J9
 U 1 1 5DE9D3E5
 P 8550 950
